Commit message: Add LiDAR mapper, RViz integration, and fix LiDAR self-occlusion
- Fix base collision cylinder blocking LiDAR (0.80m→0.60m height)
- Set LiDAR range to 8m, 720 samples, disable Gazebo visualization
- Raise furniture heights above LiDAR scan plane (0.765m) with varied heights
- Add mapper node: Bresenham ray-tracing occupancy grid on /map
- Add RViz to both launch files with fullscreen top-down mapping config
- LaserScan decay time 9999s for accumulated point cloud display
- Mapper captures RViz screenshot on finish to output/lidar_map.png
- Update APPROACH.md and CLAUDE.md with new architecture details

File: src/tidybot_description/urdf/tidybot.urdf.xacro (robot description, xacro)
@@ -77,6 +77,6 @@
          contact response at all angles (avoids box-corner blow-ups). -->
     <collision name="base_bumper">
-      <origin xyz="0 0 0.30" rpy="0 0 0"/>
-      <geometry><cylinder radius="0.35" length="0.80"/></geometry>
+      <origin xyz="0 0 0.25" rpy="0 0 0"/>
+      <geometry><cylinder radius="0.35" length="0.60"/></geometry>
     </collision>
   </link>
@@ -481,5 +481,5 @@
         <scan>
           <horizontal>
-            <samples>360</samples>
+            <samples>720</samples>
             <resolution>1.0</resolution>
             <min_angle>${-PI}</min_angle>
@@ -489,5 +489,5 @@
         <range>
           <min>0.12</min>
-          <max>10.0</max>
+          <max>8.0</max>
           <resolution>0.01</resolution>
         </range>
